File: pos project clone/pos project clone.kicad_pcb (KiCad board)
At the start: 2 copper layers, 66 x 55.7 mm, 46 parts, among them J1 JST_2mm_LiPo, J2 Conn_01x05_Socket, P1 USB_C_Plug_USB2.0, SW1 SW_Push, SW2 SW_Push, U1 LEXI-R10801D-00B, U2 MCP73831-2-OT, U3 SMN-303, U4 SMF05C, U5 GSM_ANT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

Commit message: added switch
Parts:
- added SW4: SW_SPST, Button_Switch_SMD:SW_DIP_SPSTx01_Slide_6.7x4.1mm_W6.73mm_P2.54mm_LowProfile_JPin, F.Cu at (18.2, 32.9)
- SW1, SW2: footprint Button_Switch_THT:SW_PUSH_6mm -> Button_Switch_SMD:SW_DIP_SPSTx01_Slide_6.7x4.1mm_W6.73mm_P2.54mm_LowProfile_JPin
Connections:
- D6 pad 1: VIN -> Net-(D6-K)
- D8 pad 1: VIN -> Net-(D6-K)
Routing:
- net Net-(D6-K): track 0.00 -> 25.9 mm, vias 0 -> 2
- net VIN: track 10.6 -> 26.6 mm, vias 0 -> 2
- net GND: track 44.2 -> 34.7 mm, vias 179 -> 167
