File: pos project clone/pos project clone.kicad_sch (KiCad schematic)
At the start: 46 parts, among them J1 JST_2mm_LiPo, J2 Conn_01x05_Socket, P1 USB_C_Plug_USB2.0, SW1 SW_Push, SW2 SW_Push, U1 LEXI-R10801D-00B, U2 MCP73831-2-OT, U3 SMN-303, U4 SMF05C, U5 GSM_ANT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

Commit message: added switch
Parts:
- added SW4: SW_SPST, Button_Switch_SMD:SW_DIP_SPSTx01_Slide_6.7x4.1mm_W6.73mm_P2.54mm_LowProfile_JPin, symbol Switch:SW_SPST
- SW1, SW2: footprint Button_Switch_THT:SW_PUSH_6mm -> Button_Switch_SMD:SW_DIP_SPSTx01_Slide_6.7x4.1mm_W6.73mm_P2.54mm_LowProfile_JPin
Connections:
- net VIN: now also SW4.2 (B); no longer D6.1 (K), D8.1 (K)
- new net: D6.1 (K), D8.1 (K), SW4.1 (A)
Changed lines of the file:
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@@
 	(wire
 		(pts
+			(xy 154.94 62.23) (xy 162.56 62.23)
+		)
+		(stroke
+			(width 0)
+			(type default)
+		)
+	)
+	(wire
+		(pts
 			(xy 186.69 121.92) (xy 190.5 121.92)
 		)
@@
 	(wire
 		(pts
-			(xy 154.94 72.39) (xy 144.78 72.39)
+			(xy 144.78 72.39) (xy 162.56 72.39)
 		)
 		(stroke
@@
 	(wire
 		(pts
-			(xy 154.94 63.5) (xy 154.94 72.39)
-		)
-		(stroke
-			(width 0)
-			(type default)
-		)
-	)
-	(wire
-		(pts
 			(xy 180.34 181.61) (xy 180.34 180.34)
 		)
@@
 	(symbol
 		(lib_id "power:VCC")
-		(at 154.94 63.5 0)
+		(at 154.94 62.23 0)
 		(unit 1)
 		(exclude_from_sim no)
@@
 		(fields_autoplaced yes)
 		(property "Reference" "#PWR022"
-			(at 154.94 67.31 0)
+			(at 154.94 66.04 0)
 			(effects
 				(font
@@
 		)
 		(property "Value" "VIN"
-			(at 154.94 58.42 0)
+			(at 154.94 57.15 0)
 			(effects
 				(font
@@
 		)
 		(property "Footprint" ""
-			(at 154.94 63.5 0)
+			(at 154.94 62.23 0)
 			(effects
 				(font
@@
 		)
 		(property "Datasheet" ""
-			(at 154.94 63.5 0)
+			(at 154.94 62.23 0)
 			(effects
 				(font
@@
 		)
 		(property "Description" "Power symbol creates a global label with name \"VCC\""
-			(at 154.94 63.5 0)
+			(at 154.94 62.23 0)
 			(effects
 				(font
@@
 			)
 		)
-		(property "Footprint" "Button_Switch_THT:SW_PUSH_6mm"
+		(property "Footprint" "Button_Switch_SMD:SW_DIP_SPSTx01_Slide_6.7x4.1mm_W6.73mm_P2.54mm_LowProfile_JPin"
 			(at 307.34 60.96 0)
 			(effects
@@
 			)
 		)
-		(property "Footprint" "Button_Switch_THT:SW_PUSH_6mm"
+		(property "Footprint" "Button_Switch_SMD:SW_DIP_SPSTx01_Slide_6.7x4.1mm_W6.73mm_P2.54mm_LowProfile_JPin"
 			(at 326.39 36.83 0)
 			(effects
@@
 				)
 			)
+		)
+	)
+	(symbol
+		(lib_id "Switch:SW_SPST")
+		(at 162.56 67.31 90)
+		(unit 1)
+		(exclude_from_sim no)
+		(in_bom yes)
+		(on_board yes)
+		(dnp no)
+		(fields_autoplaced yes)
+		(property "Reference" "SW4"
+			(at 163.83 66.0399 90)
+			(effects
+				(font
+					(size 1.27 1.27)
+				)
+				(justify right)
+			)
+		)
+		(property "Value" "SW_SPST"
+			(at 163.83 68.5799 90)
+			(effects
+				(font
+					(size 1.27 1.27)
+				)
+				(justify right)
+			)
+		)
+		(property "Footprint" "Button_Switch_SMD:SW_DIP_SPSTx01_Slide_6.7x4.1mm_W6.73mm_P2.54mm_LowProfile_JPin"
+			(at 162.56 67.31 0)
+			(effects
+				(font
+					(size 1.27 1.27)
+				)
+				(hide yes)
+			)
+		)
+		(property "Datasheet" "~"
+			(at 162.56 67.31 0)
+			(effects
+				(font
+					(size 1.27 1.27)
+				)
+				(hide yes)
+			)
+		)
+		(property "Description" "Single Pole Single Throw (SPST) switch"
+			(at 162.56 67.31 0)
+			(effects
+				(font
+					(size 1.27 1.27)
+				)
+				(hide yes)
+			)
+		)
+		(pin "1"
+		)
+		(pin "2"
+		)
+		(instances
+			(project ""
+				(path "/a2f47d81-8401-48b8-b89d-145d5fd985bd"
+					(reference "SW4")
+					(unit 1)
+				)
+			)
